File: hardware/matrixdriver.sch (EAGLE design)
At the start: 24 parts, among them IC1 75176AD, IC2 4017D, Q1 CSM-7X-DU

Commit message: more schematic
Parts:
- added JP1: (no value), pinhead-fixdrills:PINHD-2X8_2.54-90°
Connections:
- new net N$33: JP1.1, R9.2
- new net N$34: JP1.3, R10.2
- new net N$35: JP1.5, R11.2
- new net N$36: JP1.7, R12.2
- new net N$37: JP1.9, R13.2
- new net N$38: JP1.11, R14.2
- new net N$39: JP1.13, R15.2
- new net N$40: JP1.15, R16.2
- net N$25: now also JP1.16
Other:
- moved on the sheet: R10, R11, R12, R13, R14, R15, R16, R9
Changed lines of the file:
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@@
 <part name="IC2" library="40xx" deviceset="4017" device="D"/>
 <part name="IC3" library="uln-udn" deviceset="ULN2803A" device="SMD"/>
+<part name="JP1" library="pinhead-fixdrills" deviceset="PINHD-2X8" device="_2.54-90°"/>
 </parts>
 <sheets>
@@
 <instance part="R7" gate="G$1" x="121.92" y="86.36"/>
 <instance part="R8" gate="G$1" x="121.92" y="93.98"/>
-<instance part="R9" gate="G$1" x="136.906" y="90.424"/>
-<instance part="R10" gate="G$1" x="137.16" y="82.55"/>
-<instance part="R11" gate="G$1" x="137.16" y="75.184"/>
-<instance part="R12" gate="G$1" x="136.906" y="67.056"/>
-<instance part="R13" gate="G$1" x="136.398" y="59.69"/>
-<instance part="R14" gate="G$1" x="137.414" y="51.816"/>
-<instance part="R15" gate="G$1" x="149.606" y="47.244"/>
-<instance part="R16" gate="G$1" x="149.86" y="40.64"/>
+<instance part="R9" gate="G$1" x="137.16" y="93.98"/>
+<instance part="R10" gate="G$1" x="137.16" y="86.868"/>
+<instance part="R11" gate="G$1" x="137.668" y="79.248"/>
+<instance part="R12" gate="G$1" x="137.922" y="72.136"/>
+<instance part="R13" gate="G$1" x="138.176" y="65.278"/>
+<instance part="R14" gate="G$1" x="138.176" y="58.42"/>
+<instance part="R15" gate="G$1" x="138.43" y="51.562"/>
+<instance part="R16" gate="G$1" x="138.684" y="44.45"/>
 <instance part="Q1" gate="P" x="35.814" y="35.56" rot="R270"/>
 <instance part="IC1" gate="G$1" x="116.84" y="-15.24"/>
@@
 <instance part="IC2" gate="A" x="114.3" y="20.32"/>
 <instance part="IC3" gate="G$1" x="162.56" y="22.86"/>
+<instance part="JP1" gate="A" x="160.02" y="86.36"/>
 </instances>
 <busses>
@@
 <segment>
 <pinref part="IC3" gate="G$1" pin="O1"/>
-<wire x1="175.26" y1="33.02" x2="180.34" y2="33.02" width="0.1524" layer="91"/>
+<wire x1="175.26" y1="33.02" x2="177.8" y2="33.02" width="0.1524" layer="91"/>
+<wire x1="177.8" y1="33.02" x2="177.8" y2="76.2" width="0.1524" layer="91"/>
+<pinref part="JP1" gate="A" pin="16"/>
+<wire x1="177.8" y1="76.2" x2="165.1" y2="76.2" width="0.1524" layer="91"/>
 </segment>
 </net>
@@
 </segment>
 </net>
+<net name="N$33" class="0">
+<segment>
+<pinref part="JP1" gate="A" pin="1"/>
+<wire x1="157.48" y1="93.98" x2="142.24" y2="93.98" width="0.1524" layer="91"/>
+<pinref part="R9" gate="G$1" pin="2"/>
+</segment>
+</net>
+<net name="N$34" class="0">
+<segment>
+<pinref part="JP1" gate="A" pin="3"/>
+<wire x1="157.48" y1="91.44" x2="143.002" y2="91.44" width="0.1524" layer="91"/>
+<wire x1="142.24" y1="86.868" x2="143.002" y2="86.868" width="0.1524" layer="91"/>
+<wire x1="143.002" y1="86.868" x2="143.002" y2="91.44" width="0.1524" layer="91"/>
+<pinref part="R10" gate="G$1" pin="2"/>
+</segment>
+</net>
+<net name="N$35" class="0">
+<segment>
+<pinref part="JP1" gate="A" pin="5"/>
+<wire x1="157.48" y1="88.9" x2="143.51" y2="88.9" width="0.1524" layer="91"/>
+<wire x1="143.51" y1="88.9" x2="143.51" y2="79.248" width="0.1524" layer="91"/>
+<wire x1="143.51" y1="79.248" x2="142.748" y2="79.248" width="0.1524" layer="91"/>
+<pinref part="R11" gate="G$1" pin="2"/>
+</segment>
+</net>
+<net name="N$36" class="0">
+<segment>
+<wire x1="143.002" y1="72.136" x2="144.018" y2="72.136" width="0.1524" layer="91"/>
+<wire x1="144.018" y1="72.136" x2="144.018" y2="86.36" width="0.1524" layer="91"/>
+<pinref part="JP1" gate="A" pin="7"/>
+<wire x1="144.018" y1="86.36" x2="157.48" y2="86.36" width="0.1524" layer="91"/>
+<pinref part="R12" gate="G$1" pin="2"/>
+</segment>
+</net>
+<net name="N$37" class="0">
+<segment>
+<pinref part="JP1" gate="A" pin="9"/>
+<wire x1="157.48" y1="83.82" x2="144.526" y2="83.82" width="0.1524" layer="91"/>
+<wire x1="144.526" y1="83.82" x2="144.526" y2="65.278" width="0.1524" layer="91"/>
+<wire x1="144.526" y1="65.278" x2="143.256" y2="65.278" width="0.1524" layer="91"/>
+<pinref part="R13" gate="G$1" pin="2"/>
+</segment>
+</net>
+<net name="N$38" class="0">
+<segment>
+<pinref part="JP1" gate="A" pin="11"/>
+<wire x1="157.48" y1="81.28" x2="145.034" y2="81.28" width="0.1524" layer="91"/>
+<wire x1="145.034" y1="81.28" x2="145.034" y2="58.42" width="0.1524" layer="91"/>
+<wire x1="145.034" y1="58.42" x2="143.256" y2="58.42" width="0.1524" layer="91"/>
+<pinref part="R14" gate="G$1" pin="2"/>
+</segment>
+</net>
+<net name="N$39" class="0">
+<segment>
+<pinref part="JP1" gate="A" pin="13"/>
+<wire x1="157.48" y1="78.74" x2="145.796" y2="78.74" width="0.1524" layer="91"/>
+<wire x1="145.796" y1="78.74" x2="145.796" y2="51.562" width="0.1524" layer="91"/>
+<wire x1="145.796" y1="51.562" x2="143.51" y2="51.562" width="0.1524" layer="91"/>
+<pinref part="R15" gate="G$1" pin="2"/>
+</segment>
+</net>
+<net name="N$40" class="0">
+<segment>
+<pinref part="JP1" gate="A" pin="15"/>
+<wire x1="157.48" y1="76.2" x2="146.558" y2="76.2" width="0.1524" layer="91"/>
+<wire x1="146.558" y1="76.2" x2="146.558" y2="44.45" width="0.1524" layer="91"/>
+<wire x1="146.558" y1="44.45" x2="143.764" y2="44.45" width="0.1524" layer="91"/>
+<pinref part="R16" gate="G$1" pin="2"/>
+</segment>
+</net>

Commit message: Connect the basic elements
Parts:
- added Q2, Q3, Q4, Q5, Q6, Q7, Q8, Q9: MMBT4403LT1SMD, transistor-pnp:MMBT4403LT1SMD
Connections:
- new net N$41: Q9.B, R1.2
- new net N$42: Q8.B, R2.2
- new net N$43: Q7.B, R3.2
- new net N$44: Q6.B, R4.2
- new net N$45: Q5.B, R5.2
- new net N$46: Q4.B, R6.2
- new net N$47: Q3.B, R7.2
- new net N$48: Q2.B, R8.2
- new net N$49: Q9.C, R16.1
- new net N$50: Q8.C, R15.1
- new net N$51: Q7.C, R14.1
- new net N$52: Q6.C, R13.1
- new net N$53: Q5.C, R12.1
- new net N$54: Q4.C, R11.1
- new net N$55: Q3.C, R10.1
- new net N$56: Q2.C, R9.1
- net GND: now also U$1.GND
- net N$26: now also JP1.14
- net N$27: now also JP1.12
- net N$28: now also JP1.10
- net N$29: now also JP1.8
- net N$30: now also JP1.6
- net N$31: now also JP1.4
- net N$32: now also JP1.2
- net VCC: now also Q2.E, Q3.E, Q4.E, Q5.E, Q6.E, Q7.E, Q8.E, Q9.E, U$1.VCC
Other:
- moved on the sheet: R1, R10, R11, R12, R13, R14, R15, R16, R2, R3, R4, R5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

Commit message: first final schematic
Parts:
- added C3: (no value), rcl:CPOL-USE5-8.5
- added C4: (no value), rcl:C-EUC1206
- added IC4: 7805T, linear:7805T
- added J1: DCJ0202, con-jack:DCJ0202
- added JP2, JP3: (no value), pinhead:PINHD-1X3
- added PORTSELECT: (no value), pinhead:PINHD-2X3
- added TP1, TP2, TP3, TP4, TP5, TP6: TPSQTP20SQ, testpad:TPSQTP20SQ
Connections:
- new net N$57: IC1.A, JP2.1, JP3.1
- new net N$58: IC1.B, JP2.2, JP3.2
- new net N$59: TP5.TP, U$1.PA2(/RESET)
- new net N$60: PORTSELECT.2, U$1.(INT0)PD2
- new net N$61: PORTSELECT.4, U$1.(T1)PD5
- new net N$62: PORTSELECT.6, U$1.(ICP)PD6
- new net N$65: C3.+, IC4.VI, J1.1
- net GND: now also C3.-, C4.2, IC1.GND, IC4.GND, J1.3, JP2.3, JP3.3, PORTSELECT.1, PORTSELECT.3, PORTSELECT.5, TP6.TP
- net N$6: now also TP4.TP
- net N$7: now also TP1.TP
- net N$8: now also TP3.TP
- net VCC: now also C4.1, IC4.VO
Other:
- moved on the sheet: C1, C2, IC1, IC2, IC3, JP1, Q1, Q2, Q3, Q4, Q5, Q6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
