File: hardware/matrixdriver.sch (EAGLE design)
At the start: 35 parts, among them IC1 75176AD, IC2 4017D, IC3 ULN2803, IC4 7805DT, J1 DCJ0202, Q10 20MHZ, Q2 MMBT4403LT1SMD, Q3 MMBT4403LT1SMD, Q4 MMBT4403LT1SMD, Q5 MMBT4403LT1SMD, Q6 MMBT4403LT1SMD, Q7 MMBT4403LT1SMD, Q8 MMBT4403LT1SMD, Q9 MMBT4403LT1SMD

Commit message: working on board finalisation
Parts:
- removed C3: 100µ, rcl:CPOL-USUD-6,3X5,8
- added C6: 100UF, Panasonic-EEEFT_EEEH:EEE-HC1C101XP-CASE-D8
Connections:
- net GND: now also C6.2; no longer C3.-
- net N$65: now also C6.1; no longer C3.+
Changed lines of the file:
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@@
 <part name="JP4" library="pinhead" deviceset="PINHD-2X3" device="" value="P.SELECT"/>
 <part name="IC4" library="linear" deviceset="78*" device="DT" technology="05" value="7805DT"/>
-<part name="C3" library="rcl" deviceset="CPOL-US" device="UD-6,3X5,8" value="100µ"/>
 <part name="C4" library="rcl" deviceset="C-EU" device="C1206" value="10µ"/>
 <part name="J1" library="con-jack" deviceset="DCJ0202" device=""/>
@@
 <part name="CTS742C083_2" library="resistor-net" deviceset="CTS742C083" device="" value="1k"/>
 <part name="C5" library="resistor" deviceset="C-EU" device="C1206" value="100n"/>
+<part name="C6" library="Panasonic-EEEFT_EEEH" deviceset="EEE-" device="-CASE-D8" technology="HC1C101XP" value="100UF"/>
 </parts>
 <sheets>
@@
 <instance part="JP4" gate="A" x="48.26" y="15.24"/>
 <instance part="IC4" gate="A1" x="5.08" y="152.4" rot="R90"/>
-<instance part="C3" gate="G$1" x="7.62" y="129.54" rot="R90"/>
 <instance part="C4" gate="G$1" x="7.62" y="170.18" rot="R90"/>
 <instance part="J1" gate="G$1" x="7.62" y="104.14" rot="R90"/>
@@
 <instance part="CTS742C083_2" gate="G$1" x="101.6" y="101.6"/>
 <instance part="C5" gate="G$1" x="35.56" y="50.8" rot="R180"/>
+<instance part="C6" gate="A" x="5.08" y="134.62"/>
 </instances>
 <busses>
@@
 <wire x1="10.16" y1="111.76" x2="10.16" y2="119.38" width="0.1524" layer="91"/>
 <wire x1="10.16" y1="119.38" x2="15.24" y2="119.38" width="0.1524" layer="91"/>
-<wire x1="15.24" y1="119.38" x2="15.24" y2="129.54" width="0.1524" layer="91"/>
 <junction x="15.24" y="152.4"/>
 <pinref part="C4" gate="G$1" pin="2"/>
-<wire x1="15.24" y1="129.54" x2="15.24" y2="152.4" width="0.1524" layer="91"/>
+<wire x1="15.24" y1="119.38" x2="15.24" y2="134.62" width="0.1524" layer="91"/>
+<wire x1="15.24" y1="134.62" x2="15.24" y2="152.4" width="0.1524" layer="91"/>
 <wire x1="12.7" y1="170.18" x2="15.24" y2="170.18" width="0.1524" layer="91"/>
 <wire x1="15.24" y1="170.18" x2="15.24" y2="152.4" width="0.1524" layer="91"/>
-<pinref part="C3" gate="G$1" pin="-"/>
-<wire x1="12.7" y1="129.54" x2="15.24" y2="129.54" width="0.1524" layer="91"/>
-<junction x="15.24" y="129.54"/>
+<pinref part="C6" gate="A" pin="2"/>
+<wire x1="12.7" y1="134.62" x2="15.24" y2="134.62" width="0.1524" layer="91"/>
+<junction x="15.24" y="134.62"/>
 </segment>
 <segment>
@@
 <segment>
 <pinref part="IC4" gate="A1" pin="VI"/>
-<pinref part="C3" gate="G$1" pin="+"/>
-<wire x1="5.08" y1="142.24" x2="5.08" y2="129.54" width="0.1524" layer="91"/>
-<wire x1="5.08" y1="129.54" x2="5.08" y2="111.76" width="0.1524" layer="91"/>
-<junction x="5.08" y="129.54"/>
+<wire x1="5.08" y1="142.24" x2="5.08" y2="134.62" width="0.1524" layer="91"/>
+<wire x1="5.08" y1="134.62" x2="5.08" y2="111.76" width="0.1524" layer="91"/>
 <pinref part="J1" gate="G$1" pin="1"/>
-</segment>
-</net>
+<pinref part="C6" gate="A" pin="1"/>
+<junction x="5.08" y="134.62"/>
+</segment>
+</net>

Commit message: working on partlist
add numbers document with parts from digikey
Parts:
- removed Q10: 20MHZ, adafruit:CRYSTALHC49S
- added Q1: 20MHZ, crystal:CRYSTALHC49UP
Connections:
- net N$11: now also Q1.2; no longer Q10.2
- net N$12: now also Q1.1; no longer Q10.1
Changed lines of the file:
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@@
 <part name="J1" library="con-jack" deviceset="DCJ0202" device=""/>
 <part name="TP2" library="testpad" deviceset="TPSQ" device="TP19SQ" value="TPSQTP19SQ"/>
-<part name="Q10" library="adafruit" deviceset="CRYSTAL" device="HC49S" value="20MHZ"/>
 <part name="CTS742C083_3" library="resistor-net" deviceset="CTS742C083" device="" value="10"/>
 <part name="CTS742C083_4" library="resistor-net" deviceset="CTS742C083" device="" value="10"/>
@@
 <part name="C5" library="resistor" deviceset="C-EU" device="C1206" value="100n"/>
 <part name="C6" library="Panasonic-EEEFT_EEEH" deviceset="EEE-" device="-CASE-D8" technology="HC1C101XP" value="100UF"/>
+<part name="Q1" library="crystal" deviceset="CRYSTAL" device="HC49UP" value="20MHZ"/>
 </parts>
 <sheets>
@@
 <instance part="IC2" gate="P" x="109.22" y="73.66" rot="R90"/>
 <instance part="TP2" gate="G$1" x="60.96" y="121.92" rot="R270"/>
-<instance part="Q10" gate="G$1" x="30.48" y="68.58" rot="R90"/>
 <instance part="CTS742C083_3" gate="G$1" x="152.4" y="170.18"/>
 <instance part="CTS742C083_4" gate="G$1" x="152.4" y="96.52"/>
@@
 <instance part="C5" gate="G$1" x="35.56" y="50.8" rot="R180"/>
 <instance part="C6" gate="A" x="5.08" y="134.62"/>
+<instance part="Q1" gate="G$1" x="30.48" y="68.58" rot="R90"/>
 </instances>
 <busses>
@@
 <wire x1="30.48" y1="71.12" x2="30.48" y2="73.66" width="0.1524" layer="91"/>
 <junction x="30.48" y="73.66"/>
-<pinref part="Q10" gate="G$1" pin="2"/>
+<pinref part="Q1" gate="G$1" pin="2"/>
 </segment>
 </net>
@@
 <wire x1="30.48" y1="63.5" x2="30.48" y2="66.04" width="0.1524" layer="91"/>
 <junction x="30.48" y="63.5"/>
-<pinref part="Q10" gate="G$1" pin="1"/>
-</segment>
-</net>
+<pinref part="Q1" gate="G$1" pin="1"/>
+</segment>
+</net>

Commit message: fix some layout errors
Parts:
- removed J1: DCJ0202, con-jack:DCJ0202
- added U$2: CUI_PJ-102A, con-dc-jack:CUI_PJ-102A
Connections:
- net GND: now also U$2.VSS; no longer J1.3
- net N$65: now also U$2.VDD; no longer J1.1
Changed lines of the file:
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@@
 <part name="IC4" library="linear" deviceset="78*" device="DT" technology="05" value="7805DT"/>
 <part name="C4" library="rcl" deviceset="C-EU" device="C1206" value="10µ"/>
-<part name="J1" library="con-jack" deviceset="DCJ0202" device=""/>
 <part name="TP2" library="testpad" deviceset="TPSQ" device="TP19SQ" value="TPSQTP19SQ"/>
 <part name="CTS742C083_3" library="resistor-net" deviceset="CTS742C083" device="" value="10"/>
@@
 <part name="C6" library="Panasonic-EEEFT_EEEH" deviceset="EEE-" device="-CASE-D8" technology="HC1C101XP" value="100UF"/>
 <part name="Q1" library="crystal" deviceset="CRYSTAL" device="HC49UP" value="20MHZ"/>
+<part name="U$2" library="con-dc-jack" deviceset="CUI_PJ-102A" device=""/>
 </parts>
 <sheets>
@@
 <instance part="IC4" gate="A1" x="5.08" y="152.4" rot="R90"/>
 <instance part="C4" gate="G$1" x="7.62" y="170.18" rot="R90"/>
-<instance part="J1" gate="G$1" x="7.62" y="104.14" rot="R90"/>
 <instance part="IC2" gate="P" x="109.22" y="73.66" rot="R90"/>
 <instance part="TP2" gate="G$1" x="60.96" y="121.92" rot="R270"/>
@@
 <instance part="C6" gate="A" x="5.08" y="134.62"/>
 <instance part="Q1" gate="G$1" x="30.48" y="68.58" rot="R90"/>
+<instance part="U$2" gate="G$1" x="12.7" y="101.6" rot="R270"/>
 </instances>
 <busses>
@@
 <wire x1="12.7" y1="152.4" x2="15.24" y2="152.4" width="0.1524" layer="91"/>
 <label x="20.32" y="152.4" size="1.778" layer="95" xref="yes"/>
-<pinref part="J1" gate="G$1" pin="3"/>
 <wire x1="15.24" y1="152.4" x2="20.32" y2="152.4" width="0.1524" layer="91"/>
-<wire x1="10.16" y1="111.76" x2="10.16" y2="119.38" width="0.1524" layer="91"/>
-<wire x1="10.16" y1="119.38" x2="15.24" y2="119.38" width="0.1524" layer="91"/>
 <junction x="15.24" y="152.4"/>
 <pinref part="C4" gate="G$1" pin="2"/>
-<wire x1="15.24" y1="119.38" x2="15.24" y2="134.62" width="0.1524" layer="91"/>
+<wire x1="15.24" y1="109.22" x2="15.24" y2="134.62" width="0.1524" layer="91"/>
 <wire x1="15.24" y1="134.62" x2="15.24" y2="152.4" width="0.1524" layer="91"/>
 <wire x1="12.7" y1="170.18" x2="15.24" y2="170.18" width="0.1524" layer="91"/>
@@
 <wire x1="12.7" y1="134.62" x2="15.24" y2="134.62" width="0.1524" layer="91"/>
 <junction x="15.24" y="134.62"/>
+<pinref part="U$2" gate="G$1" pin="VSS"/>
 </segment>
 <segment>
@@
 <pinref part="IC4" gate="A1" pin="VI"/>
 <wire x1="5.08" y1="142.24" x2="5.08" y2="134.62" width="0.1524" layer="91"/>
-<wire x1="5.08" y1="134.62" x2="5.08" y2="111.76" width="0.1524" layer="91"/>
-<pinref part="J1" gate="G$1" pin="1"/>
+<wire x1="5.08" y1="134.62" x2="5.08" y2="119.38" width="0.1524" layer="91"/>
 <pinref part="C6" gate="A" pin="1"/>
 <junction x="5.08" y="134.62"/>
-</segment>
-</net>
+<pinref part="U$2" gate="G$1" pin="VDD"/>
+<wire x1="5.08" y1="119.38" x2="20.32" y2="119.38" width="0.1524" layer="91"/>
+<wire x1="20.32" y1="119.38" x2="20.32" y2="109.22" width="0.1524" layer="91"/>
+</segment>
+</net>

Commit message: resize to 5050
Connections:
- net GND: now also U$2.@3
Changed lines of the file:
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@@
 <grid distance="0.1" unitdist="inch" unit="inch" style="lines" multiple="1" display="no" altdistance="0.01" altunitdist="inch" altunit="inch"/>
 <layers>
-<layer number="1" name="Top" color="4" fill="1" visible="yes" active="no"/>
-<layer number="16" name="Bottom" color="1" fill="1" visible="yes" active="no"/>
-<layer number="17" name="Pads" color="2" fill="1" visible="yes" active="no"/>
-<layer number="18" name="Vias" color="2" fill="1" visible="yes" active="no"/>
-<layer number="19" name="Unrouted" color="6" fill="1" visible="yes" active="no"/>
-<layer number="20" name="Dimension" color="15" fill="1" visible="yes" active="no"/>
-<layer number="21" name="tPlace" color="7" fill="1" visible="yes" active="no"/>
-<layer number="22" name="bPlace" color="7" fill="1" visible="yes" active="no"/>
-<layer number="23" name="tOrigins" color="15" fill="1" visible="yes" active="no"/>
-<layer number="24" name="bOrigins" color="15" fill="1" visible="yes" active="no"/>
-<layer number="25" name="tNames" color="7" fill="1" visible="yes" active="no"/>
-<layer number="26" name="bNames" color="7" fill="1" visible="yes" active="no"/>
-<layer number="27" name="tValues" color="7" fill="1" visible="yes" active="no"/>
-<layer number="28" name="bValues" color="7" fill="1" visible="yes" active="no"/>
+<layer number="1" name="Top" color="4" fill="1" visible="no" active="no"/>
+<layer number="16" name="Bottom" color="1" fill="1" visible="no" active="no"/>
+<layer number="17" name="Pads" color="2" fill="1" visible="no" active="no"/>
+<layer number="18" name="Vias" color="2" fill="1" visible="no" active="no"/>
+<layer number="19" name="Unrouted" color="6" fill="1" visible="no" active="no"/>
+<layer number="20" name="Dimension" color="15" fill="1" visible="no" active="no"/>
+<layer number="21" name="tPlace" color="7" fill="1" visible="no" active="no"/>
+<layer number="22" name="bPlace" color="7" fill="1" visible="no" active="no"/>
+<layer number="23" name="tOrigins" color="15" fill="1" visible="no" active="no"/>
+<layer number="24" name="bOrigins" color="15" fill="1" visible="no" active="no"/>
+<layer number="25" name="tNames" color="7" fill="1" visible="no" active="no"/>
+<layer number="26" name="bNames" color="7" fill="1" visible="no" active="no"/>
+<layer number="27" name="tValues" color="7" fill="1" visible="no" active="no"/>
+<layer number="28" name="bValues" color="7" fill="1" visible="no" active="no"/>
 <layer number="29" name="tStop" color="7" fill="3" visible="no" active="no"/>
 <layer number="30" name="bStop" color="7" fill="6" visible="no" active="no"/>
@@
 <layer number="35" name="tGlue" color="7" fill="4" visible="no" active="no"/>
 <layer number="36" name="bGlue" color="7" fill="5" visible="no" active="no"/>
-<layer number="37" name="tTest" color="7" fill="1" visible="yes" active="no"/>
-<layer number="38" name="bTest" color="7" fill="1" visible="yes" active="no"/>
+<layer number="37" name="tTest" color="7" fill="1" visible="no" active="no"/>
+<layer number="38" name="bTest" color="7" fill="1" visible="no" active="no"/>
 <layer number="39" name="tKeepout" color="4" fill="11" visible="no" active="no"/>
 <layer number="40" name="bKeepout" color="1" fill="11" visible="no" active="no"/>
@@
 <layer number="44" name="Drills" color="7" fill="1" visible="no" active="no"/>
 <layer number="45" name="Holes" color="7" fill="1" visible="no" active="no"/>
-<layer number="46" name="Milling" color="3" fill="1" visible="yes" active="no"/>
-<layer number="47" name="Measures" color="7" fill="1" visible="yes" active="no"/>
-<layer number="48" name="Document" color="7" fill="1" visible="yes" active="no"/>
-<layer number="49" name="Reference" color="7" fill="1" visible="yes" active="no"/>
-<layer number="50" name="dxf" color="7" fill="1" visible="yes" active="no"/>
-<layer number="51" name="tDocu" color="7" fill="1" visible="yes" active="no"/>
-<layer number="52" name="bDocu" color="7" fill="1" visible="yes" active="no"/>
-<layer number="53" name="tGND_GNDA" color="7" fill="9" visible="yes" active="no"/>
-<layer number="54" name="bGND_GNDA" color="1" fill="9" visible="yes" active="no"/>
-<layer number="56" name="wert" color="7" fill="1" visible="yes" active="no"/>
-<layer number="57" name="tCAD" color="7" fill="1" visible="yes" active="no"/>
+<layer number="46" name="Milling" color="3" fill="1" visible="no" active="no"/>
+<layer number="47" name="Measures" color="7" fill="1" visible="no" active="no"/>
+<layer number="48" name="Document" color="7" fill="1" visible="no" active="no"/>
+<layer number="49" name="Reference" color="7" fill="1" visible="no" active="no"/>
+<layer number="50" name="dxf" color="7" fill="1" visible="no" active="no"/>
+<layer number="51" name="tDocu" color="7" fill="1" visible="no" active="no"/>
+<layer number="52" name="bDocu" color="7" fill="1" visible="no" active="no"/>
+<layer number="53" name="tGND_GNDA" color="7" fill="9" visible="no" active="no"/>
+<layer number="54" name="bGND_GNDA" color="1" fill="9" visible="no" active="no"/>
+<layer number="56" name="wert" color="7" fill="1" visible="no" active="no"/>
+<layer number="57" name="tCAD" color="7" fill="1" visible="no" active="no"/>
 <layer number="90" name="Modules" color="5" fill="1" visible="yes" active="yes"/>
 <layer number="91" name="Nets" color="2" fill="1" visible="yes" active="yes"/>
@@
 <junction x="15.24" y="152.4"/>
 <pinref part="C4" gate="G$1" pin="2"/>
-<wire x1="15.24" y1="109.22" x2="15.24" y2="134.62" width="0.1524" layer="91"/>
+<wire x1="15.24" y1="109.22" x2="15.24" y2="114.3" width="0.1524" layer="91"/>
+<wire x1="15.24" y1="114.3" x2="15.24" y2="134.62" width="0.1524" layer="91"/>
 <wire x1="15.24" y1="134.62" x2="15.24" y2="152.4" width="0.1524" layer="91"/>
 <wire x1="12.7" y1="170.18" x2="15.24" y2="170.18" width="0.1524" layer="91"/>
@@
 <junction x="15.24" y="134.62"/>
 <pinref part="U$2" gate="G$1" pin="VSS"/>
-</segment>
-<segment>
+<pinref part="U$2" gate="G$1" pin="@3"/>
+<wire x1="10.16" y1="109.22" x2="10.16" y2="114.3" width="0.1524" layer="91"/>
+<wire x1="10.16" y1="114.3" x2="15.24" y2="114.3" width="0.1524" layer="91"/>
+<junction x="15.24" y="114.3"/>
+</segment>
+<segment>

Commit message: Fix errors behind transistor
Parts:
- removed CTS742C083_1, CTS742C083_2: 1k, resistor-net:CTS742C083
- removed CTS742C083_3, CTS742C083_4: 10, resistor-net:CTS742C083
- added R1, R2, R3, R4, R5, R6, R7, R8: 1k, resistor:R-EU_R1206
- added R10, R11, R12, R13, R14, R15, R16, R9: 10, resistor:R-EU_R1206
Connections:
- removed net N$34: CTS742C083_3.7, JP1.3
- removed net N$35: CTS742C083_3.6, JP1.5
- removed net N$36: CTS742C083_3.5, JP1.7
- removed net N$56: CTS742C083_3.1, Q2.C
- new net N$44: Q2.E, R9.1
- new net N$45: Q3.E, R10.1
- new net N$46: Q5.E, R12.1
- new net N$461: C4.1, C5.2, IC1.DE, IC1.VCC, IC2P.VDD, IC4.VO, Q4.E, Q6.E, Q7.E, Q8.E, R11.1, TP2.TP, U$1.VCC
- net N$1: now also R5.1; no longer CTS742C083_2.4
- net N$13: now also R16.2; no longer CTS742C083_4.8
- net N$2: now also R6.1; no longer CTS742C083_2.3
- net N$29: now also R15.2; no longer CTS742C083_4.7
- net N$3: now also R7.1; no longer CTS742C083_2.2
- net N$30: now also R14.2; no longer CTS742C083_4.6
- net N$31: now also R13.2; no longer CTS742C083_4.5
- net N$32: now also R3.2; no longer CTS742C083_1.7
- net N$33: now also Q2.C; no longer CTS742C083_3.8
- net N$37: now also R4.2; no longer CTS742C083_1.8
- net N$38: now also R2.2; no longer CTS742C083_1.6
- net N$39: now also R1.2; no longer CTS742C083_1.5
- net N$4: now also R8.1; no longer CTS742C083_2.1
- net N$40: now also R6.2; no longer CTS742C083_2.6
- net N$41: now also R5.2; no longer CTS742C083_2.5
- net N$42: now also R8.2; no longer CTS742C083_2.8
- net N$43: now also R7.2; no longer CTS742C083_2.7
- net N$49: now also R13.1; no longer CTS742C083_4.4
- net N$5: now also R1.1; no longer CTS742C083_1.4
- net N$50: now also R14.1; no longer CTS742C083_4.3
- net N$51: now also R15.1; no longer CTS742C083_4.2
- net N$52: now also R16.1; no longer CTS742C083_4.1
- net N$53: now also JP1.7; no longer CTS742C083_3.4
- net N$54: now also JP1.5; no longer CTS742C083_3.3
- net N$55: now also JP1.3; no longer CTS742C083_3.2
- net N$6: now also R2.1; no longer CTS742C083_1.3
- net N$7: now also R3.1; no longer CTS742C083_1.2
- net N$8: now also R4.1; no longer CTS742C083_1.1
- net VCC: now also R10.2, R12.2, R9.2; no longer C4.1, C5.2, IC1.DE, IC1.VCC, IC2P.VDD, IC4.VO, Q2.E, Q3.E, Q4.E, Q5.E, Q6.E, Q7.E, Q8.E, Q9.E, TP2.TP, U$1.VCC

Commit message: fix some errors in schema
Connections:
- removed net N$52: Q6.C, R16.1
- new net N$34: Q9.E, R13.1
- new net N$35: Q7.E, R15.1
- net N$13: now also Q6.C; no longer R16.2
- net N$29: now also Q8.E, R14.1; no longer JP1.11, R15.2
- net N$30: now also Q4.E, R11.1; no longer JP1.13, R14.2
- net N$31: now also Q6.E, R16.1; no longer JP1.15, R13.2
- net N$461: no longer C4.1, C5.2, IC1.DE, IC1.VCC, IC2P.VDD, IC4.VO, Q4.E, Q6.E, Q7.E, Q8.E, R11.1, U$1.VCC
- net N$49: now also JP1.15; no longer R13.1
- net N$50: now also JP1.13; no longer R14.1
- net N$51: now also JP1.11; no longer R15.1
- net VCC: now also C4.1, C5.2, IC1.DE, IC1.VCC, IC2P.VDD, IC4.VO, R11.2, R13.2, R14.2, R15.2, R16.2, U$1.VCC
Other:
- moved on the sheet: R13, R14, R15, R16

Commit message: working on Hardware Revision 2 - fix pullup
Parts:
- added R18: 10k, resistor:R-EU_R1206
Connections:
- removed net N$461: TP2.TP
- net N$59: now also R18.1
- net VCC: now also R18.2, TP2.TP
Other:
- moved on the sheet: R1, R14, R15, R16, R2, R3, R4, R6, R7, R8
